File: LauCameraTrigger_Alchitry_Stack/LauCameraTrigger_Alchitry_Stack.kicad_pcb (KiCad board)
At the start: 2 copper layers, 55 x 45 mm, 17 parts, among them J1 DF40C-50DP (Site A / +3V3 onl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, J2 DF40C-80DP (Bank A / Site B /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, J3 DF40C-80DP (Bank B / Site C), SW1 DIP4 RGB/HV select

Commit message: LauCameraTrigger stacking board: unique JST refs + corrected order files
Rename the three JSTs to MASTER1/SLAVE1/SLAVE2 (resolving a duplicate SLAVE reference designator) so the assembly CPL has unique designators; PCB synced via F8. Regenerate production bom/bom_full/cpl from the corrected board with matched MPNs (DF40C-80DP/50DP-0.4V(51), SM07B-SRSS-TB). Matches the JLCPCB rev-1 PCBA order. FPGA Bank-B remap intentionally left uncommitted until the board is validated.

Co-Authored-By: Claude Opus 4.8 (1M context) <noreply@anthropic.com>
Parts:
- renumbered MASTER to MASTER1, SLAVE to SLAVE1, SLAVE to SLAVE2
Changed lines of the file:
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@@
 		(descr "JST SH series connector, SM07B-SRSS-TB (http://www.jst-mfg.com/product/pdf/eng/eSH.pdf)")
 		(tags "connector JST SH horizontal")
-		(property "Reference" "SLAVE"
+		(property "Reference" "SLAVE1"
 			(at 0 -3.98 90)
 			(layer "F.SilkS")
@@
 			(layers "F.Cu" "F.Mask" "F.Paste")
 			(roundrect_rratio 0.25)
-			(net "unconnected-(J5-Pin_3-Pad3)")
+			(net "unconnected-(SLAVE1-Pin_3-Pad3)")
 			(pinfunction "Pin_3_3")
 			(pintype "passive")
@@
 			(layers "F.Cu" "F.Mask" "F.Paste")
 			(roundrect_rratio 0.25)
-			(net "unconnected-(J5-Pin_5-Pad5)")
+			(net "unconnected-(SLAVE1-Pin_5-Pad5)")
 			(pinfunction "Pin_5_5")
 			(pintype "passive")
@@
 			(layers "F.Cu" "F.Mask" "F.Paste")
 			(roundrect_rratio 0.25)
-			(net "unconnected-(J5-Pin_6-Pad6)")
+			(net "unconnected-(SLAVE1-Pin_6-Pad6)")
 			(pinfunction "Pin_6_6")
 			(pintype "passive")
@@
 			(layers "F.Cu" "F.Mask" "F.Paste")
 			(roundrect_rratio 0.25)
-			(net "unconnected-(J5-Pin_7-Pad7)")
+			(net "unconnected-(SLAVE1-Pin_7-Pad7)")
 			(pinfunction "Pin_7_7")
 			(pintype "passive")
@@
 		(descr "JST SH series connector, SM07B-SRSS-TB (http://www.jst-mfg.com/product/pdf/eng/eSH.pdf)")
 		(tags "connector JST SH horizontal")
-		(property "Reference" "MASTER"
+		(property "Reference" "MASTER1"
 			(at 0 -3.98 90)
 			(layer "F.SilkS")
@@
 			(layers "F.Cu" "F.Mask" "F.Paste")
 			(roundrect_rratio 0.25)
-			(net "unconnected-(J4-Pin_6-Pad6)")
+			(net "unconnected-(MASTER1-Pin_6-Pad6)")
 			(pinfunction "Pin_6_6")
 			(pintype "passive")
@@
 			(layers "F.Cu" "F.Mask" "F.Paste")
 			(roundrect_rratio 0.25)
-			(net "unconnected-(J4-Pin_7-Pad7)")
+			(net "unconnected-(MASTER1-Pin_7-Pad7)")
 			(pinfunction "Pin_7_7")
 			(pintype "passive")
@@
 		(descr "JST SH series connector, SM07B-SRSS-TB (http://www.jst-mfg.com/product/pdf/eng/eSH.pdf)")
 		(tags "connector JST SH horizontal")
-		(property "Reference" "SLAVE"
+		(property "Reference" "SLAVE2"
 			(at 0 -3.98 90)
 			(layer "F.SilkS")
@@
 			(layers "F.Cu" "F.Mask" "F.Paste")
 			(roundrect_rratio 0.25)
-			(net "unconnected-(J6-Pin_3-Pad3)")
+			(net "unconnected-(SLAVE2-Pin_3-Pad3)")
 			(pinfunction "Pin_3_3")
 			(pintype "passive")
@@
 			(layers "F.Cu" "F.Mask" "F.Paste")
 			(roundrect_rratio 0.25)
-			(net "unconnected-(J6-Pin_5-Pad5)")
+			(net "unconnected-(SLAVE2-Pin_5-Pad5)")
 			(pinfunction "Pin_5_5")
 			(pintype "passive")
@@
 			(layers "F.Cu" "F.Mask" "F.Paste")
 			(roundrect_rratio 0.25)
-			(net "unconnected-(J6-Pin_6-Pad6)")
+			(net "unconnected-(SLAVE2-Pin_6-Pad6)")
 			(pinfunction "Pin_6_6")
 			(pintype "passive")
@@
 			(layers "F.Cu" "F.Mask" "F.Paste")
 			(roundrect_rratio 0.25)
-			(net "unconnected-(J6-Pin_7-Pad7)")
+			(net "unconnected-(SLAVE2-Pin_7-Pad7)")
 			(pinfunction "Pin_7_7")
 			(pintype "passive")

Commit message: hw: bond DIP-switch GND island to DF40 ground + document errata
The fabricated LauCameraTrigger_Alchitry_Stack had a floating GND island:
SW1 GND pads, the decoupling caps (C1/C2), and the tie-low resistor grounds
(R2/R4/R6/R8) sat on an F.Cu pour fragment never bonded to the DF40 connector
grounds. Net-level DRC missed it (all logically on GND); the RGB switches
couldn't pull their nets low and the caps were ungrounded.

Fix (PCB): explicit B.Cu GND traces from the SW1 GND pad (~140.8,99.8) to the
J3/DF40 ground region (~156.5,102.8), a GND stitching via at (162,97.5) by
C1/C2, and switch-position silkscreen (HvsV/Blue/Green/Red).

Docs (SCHEMATIC.md): new section 10 errata describing the defect, the rev-1
through-hole bodge, and the applied layout fix; flags that a fill-island is
invisible to net-level DRC (manual zone/island review + bench-test still due).

Au2.xdc intentionally left out (deferred until the new PCB rev is fab-verified).

Co-Authored-By: Claude Opus 4.8 (1M context) <noreply@anthropic.com>
Routing:
- net GND: track 0.00 -> 82.5 mm, vias 27 -> 20
- net CAM_PATTERN: track 100.5 -> 102.0 mm
- net SW_GREEN: track 29.2 -> 30.2 mm
- net CAM_TRIG: track 80.5 -> 81.5 mm
Other:
- board text added: "Blue"
- board text added: "Green"
- board text added: "HvsV"
- board text added: "Red"

Commit message: hw: populate 1k tie-high pull-ups (R1/R7) + silkscreen relabel/branding
Camera-line pull-ups for a Basler ace: the ace signal outputs (opto Line 2
and direct-coupled GPIO) are open-collector, so CAM_READY (R1) and CAM_MODE
(R7) need an external pull-up to +3V3 to read a valid logic high. Populate
R1/R7 = 1k (JLCPCB C4410 / UNI-ROYAL 1206W4F1001T5E); leave the FPGA-driven
outputs (R3/R5) and all tie-low positions DNP. Updates bom.csv, cpl.csv,
bom_full.csv, PCB/sch source (value + un-DNP), and SCHEMATIC.md rationale.

Silkscreen: relabel camera connectors to SLAVE / MASTER / SLAVE (plain silk;
unique designators MASTER1/SLAVE1/SLAVE2 kept for BOM/placement). Add
https://drhalftone.com and author "Daniel L. Lau" on front silk plus a
title block (author in company field) on the PCB and schematic.

NOTE: silkscreen changed -> gerbers/gerbers.zip are stale and must be
re-plotted in KiCad before the next fab order.

Co-Authored-By: Claude Opus 4.8 (1M context) <noreply@anthropic.com>
Parts:
- R1, R7: value 10k -> 1k
Other:
- board text added: "Daniel L. Lau"
- board text added: "https://drhalftone.com"
Changed lines of the file:
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@@
 	)
 	(paper "A4")
+	(title_block
+		(title "LauCameraTrigger_Alchitry_Stack")
+		(date "2026-07-02")
+		(company "Daniel L. Lau")
+		(comment 1 "https://drhalftone.com")
+	)
 	(layers
 		(0 "F.Cu" signal)
@@
 			(at 0 -3.98 90)
 			(layer "F.SilkS")
+			(hide yes)
+			(effects
+				(font
+					(size 1 1)
+					(thickness 0.15)
+				)
+			)
+		)
+		(fp_text user "SLAVE"
+			(at 0 -3.98 90)
+			(layer "F.SilkS")
 			(effects
 				(font
@@
 			)
 		)
-		(property "Value" "10k"
+		(property "Value" "1k"
 			(at 0 1.83 0)
 			(layer "F.Fab")
@@
 			)
 		)
-		(attr smd dnp)
+		(attr smd)
 		(duplicate_pad_numbers_are_jumpers no)
 		(fp_line
@@
 			)
 		)
-		(property "Value" "10k"
+		(property "Value" "1k"
 			(at 0 1.83 0)
 			(layer "F.Fab")
@@
 			)
 		)
-		(attr smd dnp)
+		(attr smd)
 		(duplicate_pad_numbers_are_jumpers no)
 		(fp_line
@@
 			(at 0 -3.98 90)
 			(layer "F.SilkS")
+			(hide yes)
+			(effects
+				(font
+					(size 1 1)
+					(thickness 0.15)
+				)
+			)
+		)
+		(fp_text user "MASTER"
+			(at 0 -3.98 90)
+			(layer "F.SilkS")
 			(effects
 				(font
@@
 			(at 0 -3.98 90)
 			(layer "F.SilkS")
+			(hide yes)
+			(effects
+				(font
+					(size 1 1)
+					(thickness 0.15)
+				)
+			)
+		)
+		(fp_text user "SLAVE"
+			(at 0 -3.98 90)
+			(layer "F.SilkS")
 			(effects
 				(font
@@
 		(layer "Edge.Cuts")
 	)
+	(gr_text "https://drhalftone.com"
+		(at 133 63.5 0)
+		(layer "F.SilkS")
+		(effects
+			(font
+				(size 1 1)
+				(thickness 0.15)
+			)
+			(justify left bottom)
+		)
+	)
+	(gr_text "Daniel L. Lau"
+		(at 133 66 0)
+		(layer "F.SilkS")
+		(effects
+			(font
+				(size 1 1)
+				(thickness 0.15)
+			)
+			(justify left bottom)
+		)
+	)
 	(gr_text "HvsV"
