File: LauPythonCamera_Pt_Stack/LauPythonCamera_Pt_Stack.kicad_sch (KiCad schematic)
At the start: 54 parts, among them J1 DF40C-80DP (Bank A), J2 DF40C-80DP (Bank B), J3 DF40C-50DP (Control), U1 NOIP1SN1300A-QDI, U2 AP2112K-1.8, U3 LDO 3V3 lo-noise

Commit message: fix(camera): power tree — 3.3 V ONLY. There is no 5 V on the Pt V2.
The previous rebuild assumed VDD = 5 V from USB-C, based on Alchitry's pinout page
("5V-12V board power. When plugged into USB, this can supply 5V"). That was wrong:
the Pt V2 is a 3.3 V board. Every sensor rail must come from the +3.3V on the
control header.

The VDD pins (control header, even 2-16) are now DELIBERATELY LEFT UNCONNECTED.

THE TREE
--------
  +3.3V --+--> U2  LDO 1.8 V ---------------------------> +1V8_CAM  vdd_18   80 mA
          |                                                (comes up FIRST)
          +--> U3  load switch --+-- FB1 (LOW DCR) -----> +3V3_CAM  vdd_33  140 mA
                Rds <= 50 mOhm   +-- FB2 ---------------> +3V3_PIX  vdd_pix   5 mA

U3 IS A SWITCH, NOT A REGULATOR -- and that is not a compromise, it is the only
option. You cannot LDO 3.3 V down to 3.3 V. The switch exists to SEQUENCE: the
datasheet needs vdd_18 up BEFORE vdd_33, but vdd_18 is LDO'd FROM +3.3V, so a bare
tap for vdd_33 would come up first. Something has to gate it.

FB1/FB2 ARE WHAT GIVE THE SENSOR SUPPLY REJECTION. The audit was right that a BARE
switch has no PSRR -- it passes the Pt's 4 A buck ripple and every FPGA/DDR3
transient straight into the sensor's analog domain. But the fix is a FILTER, not an
LDO: a bead + cap rolls off at -40 dB/decade, whereas an LDO's PSRR DEGRADES above
~100 kHz, which is exactly where those transients live. For the noise that actually
threatens this sensor the passive filter is the BETTER tool, not the cheaper one.
I reached for the expensive one and rebuilt the tree around a 5 V rail that does
not exist, when the real defect was a missing 20-cent filter.

FB1 MUST BE LOW-DCR (<= 50 mOhm). Hard spec. It carries 140 mA; a garden-variety
0.3 ohm bead drops 42 mV and pushes vdd_33 under its 3.2 V floor.

vdd_pix hangs off the SAME switched node, so it CANNOT outlive vdd_33. The
power-down anti-sequence stays dead -- no clamp, no diode, no supervisor. This is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
Parts:
- added C34: 100n, Capacitor_SMD:C_0402_1005Metric, symbol Device:C
- added FB2: BLM18 600R@100MHz, Inductor_SMD:L_0603_1608Metric, symbol Device:FerriteBead
- C31: value 10u (U3 Cout) -> 10u
- C32: value 10u -> 100n; footprint Capacitor_SMD:C_0805_2012Metric -> Capacitor_SMD:C_0402_1005Metric
- C33: value 100n -> 10u; footprint Capacitor_SMD:C_0402_1005Metric -> Capacitor_SMD:C_0805_2012Metric
- FB1: value BLM18 600R@100MHz -> BLM18 low-DCR <=50m
- U3: value LDO 3V3 lo-noise -> LoadSw Rds<=50m
Connections:
- net +3V3_CAM: now also FB1.2; no longer C31.1, FB1.1, U3.5 (VOUT)
- net +3V3_PIX: now also FB2.2; no longer FB1.2
- net +3V3_SYS: now also C33.1, R8.1, U2.1 (VIN), U3.1 (VIN), C34.1
- net GND: now also C34.2
- removed net VDD_SYS: C32.1, C33.1, J3.10 (C10), J3.12 (C12), J3.14 (C14), J3.16 (C16), J3.2 (C2), J3.4 (C4), J3.6 (C6), J3.8 (C8), R8.1, U2.1 (VIN), U3.1 (VIN)
- new net +3V3_SW: C31.1, C32.1, FB1.1, FB2.1, U3.5 (VOUT)
- no-connect marks 101 -> 109

Commit message: fix(camera): REBUILD the power tree — boost + LDO. The 3.3 V tap never worked.
The Pt V2's +3V3 rail is 3.278 V, not 3.300 V. It is fully derivable from
Alchitry's own schematic: the ADP5052 buck ch.1 divider (R16 31.6k / R15 10.2k)
against an 0.8 V feedback reference. Validated — the same convention predicts
the Pt's 1V, 1V8 and 1V35 rails exactly. With the ADP5052's +/-1.5 % accuracy
the rail is 3.229 to 3.327 V.

Three consequences, all arithmetic, none of them opinion:

  * vdd_pix (3.25-3.35 V) is OUT OF SPEC at the low corner, by 21 mV.
  * vdd_33 had ~7 mV of worst-case margin after ferrite + connector IR drop.
  * The tap made correct power-up sequencing IMPOSSIBLE. vdd_33 tapped from
    +3V3 rises the instant the Pt's rail does, but 1.8 V can only be made by
    LDO'ing down from that same rail — and an LDO's output cannot precede its
    input. So vdd_18 always came up AFTER vdd_33: the order the datasheet
    explicitly forbids, on every power-up, by construction. That risks latch-up
    and a dead sensor. No ferrite or load switch downstream can fix it.

New tree: +3V3 -> TPS61023 boost -> 4.46 V -> two TPS7A2033 LDOs (vdd_33,
vdd_pix); vdd_18 from a TPS7A2018 off +3V3 directly. The boost is not the
regulator — it exists only to give the LDOs headroom, because you cannot LDO
3.278 V down to an accurate 3.300 V. All accuracy and all noise rejection
(75-95 dB PSRR vs the FPGA's buck ripple) happen in the LDOs.

Sequencing is now structural, not a race between time constants. TWO TLV803S
supervisors are required, not one: a single open-drain driving both enable
nodes couples them together whenever RESET is released, dragging EN_PIX above
its 0.9 V threshold and bringing vdd_pix up alongside vdd_33. Resistors cannot
fix it (decoupling and pull-down demand opposite values) and a diode-AND cannot
either (Schottky leakage falsely enables; silicon Vf exceeds the 0.3 V
EN-low max). U6 gates vdd_pix, its pull-up tied to vdd_33 so vdd_pix physically
cannot enable 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
Parts:
- removed C25: 10u, Capacitor_SMD:C_0805_2012Metric, symbol Device:C
- removed FB1: BLM18 low-DCR <=50m, Inductor_SMD:L_0603_1608Metric, symbol Device:FerriteBead
- removed FB2: BLM18 600R@100MHz, Inductor_SMD:L_0603_1608Metric, symbol Device:FerriteBead
- removed U3: LoadSw Rds<=50m, Package_TO_SOT_SMD:SOT-23-5, symbol LauSensors:REG_5PIN_EN
- added C35, C36, C37: 1u, Capacitor_SMD:C_0402_1005Metric, symbol Device:C
- added C38, C40: 100n, Capacitor_SMD:C_0402_1005Metric, symbol Device:C
- added C39: 10n, Capacitor_SMD:C_0402_1005Metric, symbol Device:C
- added C41: 220n, Capacitor_SMD:C_0402_1005Metric, symbol Device:C
- added L1: 2.2uH, Inductor_SMD:L_Sunlord_SWPA3012S, symbol Device:L
- added R15, R16: 100k, Resistor_SMD:R_0402_1005Metric, symbol Device:R
- added R17: 1k, Resistor_SMD:R_0402_1005Metric, symbol Device:R
- added U3: TPS61023DRLR, Package_SON:SOT-563, symbol LauSensors:BOOST_TPS61023
- added U4, U5: TPS7A2033PDBVR, Package_TO_SOT_SMD:SOT-23-5, symbol LauSensors:REG_5PIN_EN
- added U6, U7: TLV803SDBZT, Package_TO_SOT_SMD:SOT-23, symbol LauSensors:SUPERVISOR_TLV803
- C10, C11, C8, C9: value 1u -> 100n
- C29, C30, C34: value 100n -> 1u
- C32: value 100n -> 10u; footprint Capacitor_SMD:C_0402_1005Metric -> Capacitor_SMD:C_0805_2012Metric
- R8: value 10k -> 649k
- R9: value 10k -> 100k
- U2: value AP2112K-1.8 -> TPS7A2018PDBVR
Connections:
- net +1V8_CAM: now also C30.1, U4.3 (EN); no longer R9.1
- net +3V3_CAM: now also C35.1, R15.1, U4.5 (VOUT)
- net +3V3_PIX: now also C37.1, U5.5 (VOUT)
- net +3V3_SYS: now also C29.1, C31.1, U2.3 (EN), C38.1, C40.1, L1.1, R16.1, U3.3 (VIN), U6.3 (VDD), U7.3 (VDD); no longer C33.1, C34.1, R8.1
- net GND: now also R9.2, C35.2, C36.2, C37.2, C38.2, C39.2, C40.2, C41.2, U3.4 (GND), U4.2 (GND), U5.2 (GND), U6.1 (GND), U7.1 (GND)
- net +3V3_SW renamed +4V5
- net +4V5: now also C33.1, C34.1, R8.1, C36.1, U3.6 (VOUT), U4.1 (VIN), U5.1 (VIN); no longer C31.1
- removed net SEQ_1V8: C29.1, R8.2, U2.3 (EN)
- removed net SEQ_3V3: C30.1, R9.2
- new net EN_BOOST: C41.1, R17.2, U3.2 (EN)
- new net EN_PIX: C39.1, R15.2, U5.3 (EN), U6.2 (RESET)
- new net FB_BOOST: R8.2, R9.1, U3.1 (FB)
- new net RST_BOOST: R16.2, R17.1, U7.2 (RESET)
- new net SW: L1.2, U3.5 (SW)
- no-connect marks 109 -> 110

Commit message: fix(camera): footprints — every one now resolves. Two were broken, two were missing.
Verified all 10 footprint references in the schematic against the authoritative
sources rather than trusting the names. KiCad is not installed on this machine,
so the standard names were checked against the official KiCad/kicad-footprints
repository on GitHub.

Two were WRONG and would have failed to resolve:

  * U3 (boost) was "Package_SON:SOT-563". SOT-563 lives in Package_TO_SOT_SMD,
    not Package_SON. Fixed.
  * J1/J2/J3 referenced "Connector_Hirose_DF40:...". THAT LIBRARY DOES NOT EXIST
    in KiCad -- the real one is Connector_Hirose, and it ships no DF40 parts.
    The fabbed LauCameraTrigger_Alchitry_Stack board used the same (nonexistent)
    library name, so it must have resolved from some machine-local library that
    is not in this repo.

Two were MISSING entirely:

  * The DF40 footprints are now vendored into LauCamera.pretty, extracted from
    the EMBEDDED definitions in the fabbed LauCameraTrigger_Alchitry_Stack
    .kicad_pcb. That is manufactured, proven geometry -- the best available
    source. Pad counts check out: 80+4 mounting posts, 50+4.
  * L1's inductor footprint did not exist in any library. Created
    L_Sunlord_SWPA3012S_3.0x3.0mm from Sunlord's own recommended land pattern
    (SWPA series datasheet, rev 2022/05/15): pads 0.8 x 1.5 mm, overall span
    C = 2.7 mm (centres +/-0.95 mm), body 3.0 x 3.0 x 1.2 mm.

The project is now self-contained: the 4 project-specific footprints live in
LauCamera.pretty, and the other 5 are KiCad standard parts confirmed to exist
upstream (C_0402, C_0805, R_0402, SOT-23, SOT-23-5, SOT-563).

Pad numbering verified against the symbols: socket 1..48, DF40s 1..80 / 1..50,
inductor 1..2. All files parse with balanced s-expressions.

Co-Authored-By: Claude Opus 4.8 (1M context) <noreply@anthropic.com>
Parts:
- J1, J2: footprint Connector_Hirose_DF40:Hirose_DF40C-80DP-0.4V_2x40-1MP_P0.4mm -> LauCamera:Hirose_DF40C-80DP-0.4V_2x40-1MP_P0.4mm
- J3: footprint Connector_Hirose_DF40:Hirose_DF40C-50DP-0.4V_2x25-1MP_P0.4mm -> LauCamera:Hirose_DF40C-50DP-0.4V_2x25-1MP_P0.4mm
- L1: footprint Inductor_SMD:L_Sunlord_SWPA3012S -> LauCamera:L_Sunlord_SWPA3012S_3.0x3.0mm
- U3: footprint Package_SON:SOT-563 -> Package_TO_SOT_SMD:SOT-563
Changed lines of the file:
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@@
 		(property "Value" "DF40C-80DP (Bank A)" (at 472.54 261.27 0)
 			(effects (font (size 1.27 1.27)) (justify left) ))
-		(property "Footprint" "Connector_Hirose_DF40:Hirose_DF40C-80DP-0.4V_2x40-1MP_P0.4mm" (at 470.0 260.0 0)
+		(property "Footprint" "LauCamera:Hirose_DF40C-80DP-0.4V_2x40-1MP_P0.4mm" (at 470.0 260.0 0)
 			(effects (font (size 1.27 1.27)) (hide yes)))
 		(pin "1")
@@
 		(property "Value" "DF40C-80DP (Bank B)" (at 642.54 261.27 0)
 			(effects (font (size 1.27 1.27)) (justify left) ))
-		(property "Footprint" "Connector_Hirose_DF40:Hirose_DF40C-80DP-0.4V_2x40-1MP_P0.4mm" (at 640.0 260.0 0)
+		(property "Footprint" "LauCamera:Hirose_DF40C-80DP-0.4V_2x40-1MP_P0.4mm" (at 640.0 260.0 0)
 			(effects (font (size 1.27 1.27)) (hide yes)))
 		(pin "1")
@@
 		(property "Value" "DF40C-50DP (Control)" (at 802.54 221.27 0)
 			(effects (font (size 1.27 1.27)) (justify left) ))
-		(property "Footprint" "Connector_Hirose_DF40:Hirose_DF40C-50DP-0.4V_2x25-1MP_P0.4mm" (at 800.0 220.0 0)
+		(property "Footprint" "LauCamera:Hirose_DF40C-50DP-0.4V_2x25-1MP_P0.4mm" (at 800.0 220.0 0)
 			(effects (font (size 1.27 1.27)) (hide yes)))
 		(pin "1")
@@
 		(property "Value" "TPS61023DRLR" (at 142.54 431.27 0)
 			(effects (font (size 1.27 1.27)) (justify left)))
-		(property "Footprint" "Package_SON:SOT-563" (at 140 430 0)
+		(property "Footprint" "Package_TO_SOT_SMD:SOT-563" (at 140 430 0)
 			(effects (font (size 1.27 1.27)) (hide yes)))
 		(pin "1")
@@
 		(property "Value" "2.2uH" (at 242.54 431.27 0)
 			(effects (font (size 1.27 1.27)) (justify left)))
-		(property "Footprint" "Inductor_SMD:L_Sunlord_SWPA3012S" (at 240 430 0)
-			(effects (font (size 1.27 1.27)) (hide yes)))
-		(pin "1")
+		(property "Footprint" "LauCamera:L_Sunlord_SWPA3012S_3.0x3.0mm" (at 240 430 0)
+			(effects (font (size 1.27 1.27)) (hide yes)))
+		(pin "1")

Commit message: fix(camera): LDO stability caps 0402 -> 0603 (DC-bias derating)
The six LDO input/output caps (C29, C30, C34-C37) were 1uF in an 0402. At the
3.3-4.5 V bias they actually see, an 0402 X7R loses 30-40% of its capacitance,
which can drop below the TPS7A20's 1 uF MINIMUM FOR STABILITY. CAMERA_POWER_DESIGN.md
specifies 0603 for exactly this reason; the schematic did not match. Now it does.

Sensor per-pin decoupling (C1-C7) stays 0402 -- those are decoupling caps, not
stability-critical, and derating there is harmless.

Full audit against the design docs also confirms:
  * all 48 sensor pins connected
  * all 8 sensor CMOS inputs have pulls, correct polarity (ss_n UP to the
    sensor's own +3V3_CAM; reset_n and trigger0-2 DOWN, fail-safe)
  * R2 = 100R differential termination on CAM_LVDSCLK -- the one pair the FPGA
    drives INTO the sensor (the other six are terminated by the FPGA's DIFF_TERM)
  * R1 = 47k ibias_master to gnd_33
  * VBSEL_A strapped high

Co-Authored-By: Claude Opus 4.8 (1M context) <noreply@anthropic.com>
Parts:
- C29, C30, C34, C35, C36, C37: footprint Capacitor_SMD:C_0402_1005Metric -> Capacitor_SMD:C_0603_1608Metric
Changed lines of the file:
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@@
 		(property "Value" "1u" (at 102.54 351.27 0)
 			(effects (font (size 1.27 1.27)) (justify left)))
-		(property "Footprint" "Capacitor_SMD:C_0402_1005Metric" (at 100 350 0)
+		(property "Footprint" "Capacitor_SMD:C_0603_1608Metric" (at 100 350 0)
 			(effects (font (size 1.27 1.27)) (hide yes)))
 		(pin "1")
@@
 		(property "Value" "1u" (at 202.54 351.27 0)
 			(effects (font (size 1.27 1.27)) (justify left)))
-		(property "Footprint" "Capacitor_SMD:C_0402_1005Metric" (at 200 350 0)
+		(property "Footprint" "Capacitor_SMD:C_0603_1608Metric" (at 200 350 0)
 			(effects (font (size 1.27 1.27)) (hide yes)))
 		(pin "1")
@@
 		(property "Value" "1u" (at 522.54 351.27 0)
 			(effects (font (size 1.27 1.27)) (justify left)))
-		(property "Footprint" "Capacitor_SMD:C_0402_1005Metric" (at 520 350 0)
+		(property "Footprint" "Capacitor_SMD:C_0603_1608Metric" (at 520 350 0)
 			(effects (font (size 1.27 1.27)) (hide yes)))
 		(pin "1")
@@
 		(property "Value" "1u" (at 622.54 351.27 0)
 			(effects (font (size 1.27 1.27)) (justify left)))
-		(property "Footprint" "Capacitor_SMD:C_0402_1005Metric" (at 620 350 0)
+		(property "Footprint" "Capacitor_SMD:C_0603_1608Metric" (at 620 350 0)
 			(effects (font (size 1.27 1.27)) (hide yes)))
 		(pin "1")
@@
 		(property "Value" "1u" (at 522.54 431.27 0)
 			(effects (font (size 1.27 1.27)) (justify left)))
-		(property "Footprint" "Capacitor_SMD:C_0402_1005Metric" (at 520 430 0)
+		(property "Footprint" "Capacitor_SMD:C_0603_1608Metric" (at 520 430 0)
 			(effects (font (size 1.27 1.27)) (hide yes)))
 		(pin "1")
@@
 		(property "Value" "1u" (at 622.54 431.27 0)
 			(effects (font (size 1.27 1.27)) (justify left)))
-		(property "Footprint" "Capacitor_SMD:C_0402_1005Metric" (at 620 430 0)
-			(effects (font (size 1.27 1.27)) (hide yes)))
-		(pin "1")
+		(property "Footprint" "Capacitor_SMD:C_0603_1608Metric" (at 620 430 0)
+			(effects (font (size 1.27 1.27)) (hide yes)))
+		(pin "1")
