File: LauPythonCamera_Pt_Stack/LauPythonCamera_Pt_Stack.kicad_sch (KiCad schematic)
At the start: 68 parts, among them J1 DF40C-80DP (Bank A), J2 DF40C-80DP (Bank B), J3 DF40C-50DP (Control), U1 NOIP1SN1300A-QDI, U2 TPS7A2018PDBVR, U3 TPS61023DRLR, U4 TPS7A2033PDBVR, U5 TPS7A2033PDBVR, U6 TLV803SDBZT, U7 TLV803SDBZT

Commit message: feat(camera): dual-source the inductor; document why every Extended part is forced
TWO ASKS: don't burn money on Extended parts, and don't leave me picking
replacements later. Addressed both.

=== The BOM is already at the Extended floor ===

JLCPCB charges ~$3 per unique EXTENDED part; BASIC parts are free. All 13
passive line items are Basic (that alone avoids ~$39). The 7 Extended parts are
each forced -- there is no Basic part that does the job:

  * TPS7A2033 (LDO 3.3 V) -- Basic has only AMS1117 / XC6206, +/-2% or worse.
    +/-2% of 3.3 V spans 3.234-3.366 V against a vdd_pix window of 3.250-3.350 V.
    They FAIL THE SPEC ON THEIR OWN, before a single millivolt of IR drop.
  * TPS7A2018 (LDO 1.8 V) -- Basic has NO 1.8 V LDO at all (3.3 V and 5 V only).
  * TLV803S (supervisor) -- Basic has NO supervisor of any kind.
  * TPS61023 (boost) -- both Basic boosts fail. TPS61040: 350 mA switch limit vs
    our 620 mA peak; it cannot deliver the load. FP6291: enough current, but
    ASYNCHRONOUS WITH NO TRUE DISCONNECT -- disabled, its output stays tied to
    the input through the inductor and Schottky, which during the supervisor's
    200 ms delay would bring vdd_33 and vdd_pix up at ~2.9 V (out of spec)
    instead of leaving them at zero. TPS61023's true disconnect is precisely
    what makes the power-up clean.
  * Inductor -- Basic has NO power inductor >= 1 uH, only 0603/0805 chip parts
    that saturate below our 620 mA peak.
  * DF40C-80DP / 50DP -- the mating connector. No substitute exists.

~$21 in feeder fees, and that is what buys a pixel supply that is in spec.

=== The inductor is now dual-sourced, so no future replacement decision ===

The Sunlord SWPA3012 had only ~1,330 stock -- exactly the part that would have
forced a substitution later. Swapped the PRIMARY to CENKER CKCS3015-2.2uH/M
(C354563), which is better on every axis: Isat 1.6 A (was 1.2 A), DCR 60 mohm
(was 98 mohm), ~3,500 stock, magnetically shielded, same 3x3 mm, same price.
Peak cur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
Parts:
- L1: footprint LauCamera:L_Sunlord_SWPA3012S_3.0x3.0mm -> LauCamera:L_Power_3x3mm_SWPA3012_CKCS3015; LCSC C36402 -> C354563; MPN SWPA3012S2R2MT -> CKCS3015-2.2uH/M
Changed lines of the file:
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@@
 		(property "Value" "2.2uH" (at 242.54 431.27 0)
 			(effects (font (size 1.27 1.27)) (justify left)))
-		(property "Footprint" "LauCamera:L_Sunlord_SWPA3012S_3.0x3.0mm" (at 240 430 0)
+		(property "Footprint" "LauCamera:L_Power_3x3mm_SWPA3012_CKCS3015" (at 240 430 0)
 			(effects (font (size 1.27 1.27)) (hide yes)))
-		(property "MPN" "SWPA3012S2R2MT" (at 240 430 0)
+		(property "MPN" "CKCS3015-2.2uH/M" (at 240 430 0)
 			(effects (font (size 1.27 1.27)) (hide yes)))
-		(property "LCSC" "C36402" (at 240 430 0)
+		(property "LCSC" "C354563" (at 240 430 0)
 			(effects (font (size 1.27 1.27)) (hide yes)))
 		(pin "1")

Commit message: fix(camera): SPICE found a real bug — L1 saturates on every startup. Resized 3x3 -> 4x4.
Simulated the power tree in LTspice with TI's ACTUAL PSpice models: TPS7A20
(SBVM961) x3, TLV803S (SBVM034) x2, TPS61023 (SLVMD68). The sensor has no public
SPICE model (confirmed with onsemi) so it is modelled as its datasheet loads plus
the board's real decoupling.

=== THE BUG SPICE FOUND ===

Peak inductor current at STARTUP is 1.496 A -- about 3x the 0.54 A steady-state
peak. It is the boost charging its output caps against its own 3.7 A internal
current limit. NOT a numerical spike: the current sits above 1.2 A for 15 us and
above 1.4 A for 6 us, on EVERY power-up.

I had sized L1 on steady-state current. Both inductors I chose were wrong:

    Sunlord SWPA3012   Isat 1.2 A  -> 0.80x   SATURATES EVERY STARTUP
    CENKER  CKCS3015   Isat 1.6 A  -> 1.07x   no margin
    SXN     SMNR4020   Isat 3.4 A  -> 2.27x   OK   <-- now fitted

Reducing the boost output cap does NOT fix it (22 uF -> 12 uF moved the peak only
1.496 -> 1.454 A). The inrush is set by the converter's soft-start, not the caps.
The inductor has to be sized for it.

L1 = SMNR4020-2.2UH (LCSC C135262): 2.2uH, Isat 3.4 A, DCR 46 mohm (better than
both previous parts), 4x4x2 mm, and 107,410 in stock -- which also kills the
"will I have to pick a replacement later" risk. New footprint built from SXN's
own land pattern (F=0.95, G=2.1, H=3.3).

=== WHAT ELSE SPICE CONFIRMED ===

Sequencing PASSES in both directions, with real TI models:
  power-up   vdd_18 (0.99ms) -> vdd_33 (211.65ms) -> vdd_pix (212.26ms)  gap 601us
  power-down vdd_pix (261.29ms) -> vdd_33 (262.07ms) -> vdd_18 (265.77ms) gap 777us
Every gap is 60-380x the required 10 us.

Steady-state rails all in spec:
  vdd_18  1.7945 V  (1.70-1.90)
  vdd_33  3.2901 V  (3.20-3.40)
  vdd_pix 3.2998 V  (3.25-3.35)  <-- dead centre of the tight window

Inrush does NOT cause a startup lockup: with a pessimistic 50 mohm source
impedance the boost droops +3V3 to 3.203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
Parts:
- L1: footprint LauCamera:L_Power_3x3mm_SWPA3012_CKCS3015 -> LauCamera:L_Power_4x4mm_SMNR4020; LCSC C354563 -> C135262; MPN CKCS3015-2.2uH/M -> SMNR4020-2.2UH
Changed lines of the file:
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@@
 		(property "Value" "2.2uH" (at 242.54 431.27 0)
 			(effects (font (size 1.27 1.27)) (justify left)))
-		(property "Footprint" "LauCamera:L_Power_3x3mm_SWPA3012_CKCS3015" (at 240 430 0)
+		(property "Footprint" "LauCamera:L_Power_4x4mm_SMNR4020" (at 240 430 0)
 			(effects (font (size 1.27 1.27)) (hide yes)))
-		(property "MPN" "CKCS3015-2.2uH/M" (at 240 430 0)
+		(property "MPN" "SMNR4020-2.2UH" (at 240 430 0)
 			(effects (font (size 1.27 1.27)) (hide yes)))
-		(property "LCSC" "C354563" (at 240 430 0)
+		(property "LCSC" "C135262" (at 240 430 0)
 			(effects (font (size 1.27 1.27)) (hide yes)))
 		(pin "1")

Commit message: fix(camera): socket P/N confirmed from onsemi's own headboard BOM — it needs the "-1"
Pulled onsemi's NOIP-48PIN-HEAD-BD-A-GEVK headboard schematic and read their BOM
(31000040 REV4). Against the NOIP1SN1300A they list:

    MFG Part#:  680-48-SM-G10-R14-1
    MFG:        ANDON SOCKET
    Count: 1    Ref: U6

So the socket already in this design is the right one -- but the part number was
MISSING THE "-1" SUFFIX. Every distributor lists it with the -1; we had
680-48-SM-G10-R14. Fixed in the schematic and the BOM.

Also confirmed OPEN-TOP, which the lens requires: the same schematic notes "U6A
Socket Cap is NOT USED for 48 Pin Socket Assembly" -- the cap/spacer belongs only
to the 84-pin PYTHON 5MP socket (686-84A-SM-G10-L14-1).

BONUS FINDING -- onsemi's own reference design independently validates our power
architecture. Their headboard powers this same sensor with a CS51414 BUCK feeding
THREE NCP3335 LDOs: -330 (3.3 V), -180 (1.8 V), and -ADJ (ADJUSTABLE). That is a
switcher making an intermediate rail, then LDOs, with a SEPARATE, TRIMMABLE
regulator for the pixel supply.

That is structurally what CAMERA_POWER_DESIGN.md §3 arrives at from first
principles -- and it is nothing like the ferrite tap the old design used. The
sensor vendor's own board does not tap a noisy rail through a bead either.

Sourcing reality: no distributor stocks the socket off the shelf. Andon direct, or
brokers (Perfect Parts, GlobalTek), both RFQ, ~70 units visible in total. Buy spares.

Co-Authored-By: Claude Opus 4.8 (1M context) <noreply@anthropic.com>
Parts:
- U1: MPN 680-48-SM-G10-R14 -> 680-48-SM-G10-R14-1
Changed lines of the file:
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@@
 		(property "Footprint" "LauCamera:Andon_680-48-SM-G10-R14" (at 170.0 120.0 0)
 			(effects (font (size 1.27 1.27)) (hide yes)))
-		(property "MPN" "680-48-SM-G10-R14" (at 170.0 120.0 0)
+		(property "MPN" "680-48-SM-G10-R14-1" (at 170.0 120.0 0)
 			(effects (font (size 1.27 1.27)) (hide yes)))
 		(property "LCSC" "" (at 170.0 120.0 0)
