File: LauPythonCamera_Pt_Stack/LauPythonCamera_Pt_Stack.kicad_pcb (KiCad board)
At the start: 4 copper layers, 55 x 45 mm, 68 parts, among them J1 DF40C-80DP (Bank A), J2 DF40C-80DP (Bank B), J3 DF40C-50DP (Control), U1 NOIP1SN1300A-QTI, U2 TPS7A2018PDBVR, U3 TPS61023DRLR, U4 TPS7A2033PDBVR, U5 TPS7A2033PDBVR, U6 TLV803SDBZT, U7 TLV803SDBZT

Commit message: fix(camera): close the two power-integrity defects -- boost hot loop + sensor decoupling
Board re-reviewed from the .kicad_pcb rather than from section 14's text, which
surfaced a defect section 14 never mentioned and outranked everything on its list.
Every figure below is measured, and DRC is clean after each step:
0 errors, 0 unconnected, 110 benign parity warnings.

A1 -- THE BOOST HAD NO OUTPUT CAPACITOR (new finding).
U3.6 (+4V5 out) was 9.81 mm from the nearest +4V5 cap, ~11.2 mm routed with a
layer change mid-path. That is the hot loop of a boost converter: the loop where
inductor current commutates into COUT every switching cycle. C32/C33 were sitting
in the middle of a wire, helping neither end -- both LDOs already have their own
input caps (C34 2.93 mm, C36 3.76 mm). Moved C32 hard against U3.6/U3.4 (2.52 mm)
with a GND via 1.59 mm from its ground pad, and C33 behind it. Loop is now ~4.6 mm
of trace plus two via transitions.

A2 -- FIVE OF U1'S ELEVEN SUPPLY PINS WERE UNDECOUPLED.
Not a schematic omission: the rails carry exactly one 1uF + one 10nF per supply
pin (C1-C4 + C12-C15 for four +3V3_CAM pins; C5-C7 + C16-C18 for three +1V8_CAM
pins). The layout had stacked all of them in a column west of the socket, which
served the two west pins and left the east/north pins on 14-24 mm runs. +3V3_PIX
scores 2.75-2.90 mm on all four of its pins -- same board, same day, done right --
which is what made the distribution diagnosis unambiguous.

Redistributed one pair per pin, no parts added, no schematic change, no BOM change:

  pin    rail    before    power side    ground side
  19     3.3V    23.4 mm      3.3 mm        1.54 mm
  22     1.8V    23.4 mm      3.3 mm        1.57 mm
  26     1.8V    23.7 mm      2.9 mm        0.49 mm
  29     3.3V    23.4 mm      2.3 mm        0.51 mm
  36     3.3V    14.0 mm      2.6 mm        0.46 mm

Caps went to B.Cu directly under the pads (verified free; bottom side already
assembles for J1-J3 and R2). Each pin got its own fee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
Parts:
- C1, C12, C13, C15, C16, C17, C2, C3, C5, C6: moved to B.Cu
- moved C15 26.0 mm to (145.0, 87.1)
- moved C2 23.8 mm to (142.7, 87.1)
- moved C16 23.4 mm to (142.9, 80.0)
- moved C5 23.4 mm to (144.8, 80.0)
- moved C12 23.0 mm to (142.9, 77.9), turned to -90 degrees
- moved C1 23.0 mm to (144.8, 77.9), turned to -90 degrees
- moved C6 22.6 mm to (145.1, 85.0), turned to -90 degrees
- moved C17 22.3 mm to (142.7, 85.0), turned to -90 degrees
- moved C13 15.5 mm to (136.0, 75.1), turned to 180 degrees
- moved C3 14.0 mm to (136.0, 73.1), turned to 180 degrees
- moved C32 6.65 mm to (110.9, 71.3), turned to 0 degrees
- moved C33 4.20 mm to (116.1, 72.5)
Routing:
- net GND: track 443.4 -> 463.7 mm, vias 40 -> 49
- net +1V8_CAM: track 76.4 -> 66.5 mm, vias 0 -> 2
- net +3V3_CAM: track 104.5 -> 98.9 mm, vias 7 -> 9
- net +4V5: track 48.2 -> 44.4 mm
- net +3V3_SYS: track 92.8 -> 91.5 mm

Commit message: feat(camera): add bring-up test points; fan the J3 power entry; drop LVDS stitching
TEST POINTS -- six 1.5 mm exposed pads (TP1-TP6), which the board had none of.

  TP1 SYS  +3V3_SYS  (111.60, 101.00)
  TP2 4V5  +4V5      (121.40,  67.50)
  TP3 1V8  +1V8_CAM  (117.30,  86.48)
  TP4 3V3  +3V3_CAM  (115.36,  88.81)
  TP5 PIX  +3V3_PIX  (128.14,  65.71)
  TP6 GND  GND       (119.64,  82.79)

Each pad is placed directly ON its rail's existing F.Cu copper, so it is connected
by overlap -- no stub, no routing, nothing to mis-wire. Positions were found by
searching along each rail's own traces for a spot where a 1.5 mm pad clears every
other net, the board edge and the socket keep-out.

They are BOARD-ONLY BY DESIGN: each carries exclude_from_bom and
exclude_from_pos_files, so they never reach JLCPCB's BOM or placement file. No
LCSC part number needed and no do-not-place instruction like U1. Footprint added
to LauCamera.pretty so the library-parity check passes.

Why they exist: CAMERA_POWER_DESIGN.md's tree has only ever been validated in
SPICE. On arrival vdd_18 must be shown to rise BEFORE vdd_33 and vdd_pix must sit
in 3.25-3.35 V -- a two-probe, scope-triggered measurement taken during power-up.
TP3 and TP4 are 3.1 mm apart with TP6 5 mm away, so that is now a hands-free
setup instead of holding two fine probes on 0402 pads beside a socket that will
hold a 27-week-lead sensor.

J3 POWER ENTRY -- fanned. Each of the eight power pins now has its own ~1.5 mm
stub to a common bus instead of current threading pad-to-pad along the 0.4 mm
pitch row. Widths left at 0.2 mm by author's decision; the shared bus/riser
carries ~320 mA against ~0.5 A for 0.2 mm on 1 oz outer copper.

Correction recorded: the earlier widening in 1935ba6 put 0.8 mm on the branch to
U3.3, which carries only the boost IC's own bias current. In a boost the input
current flows +3V3_SYS -> L1 -> SW; that branch is the 0.5 mm run east to
(113.8, 76.15) and is adequately sized.

LVDS RETURN-PATH STITCHING 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
Parts:
- added TP1: SYS, LauCamera:TestPoint_Pad_D1.5mm, F.Cu at (111.6, 101.0)
- added TP2: 4V5, LauCamera:TestPoint_Pad_D1.5mm, F.Cu at (121.4, 67.5)
- added TP3: 1V8, LauCamera:TestPoint_Pad_D1.5mm, F.Cu at (117.3, 86.5)
- added TP4: 3V3, LauCamera:TestPoint_Pad_D1.5mm, F.Cu at (115.4, 88.8)
- added TP5: PIX, LauCamera:TestPoint_Pad_D1.5mm, F.Cu at (128.1, 65.7)
- added TP6: GND, LauCamera:TestPoint_Pad_D1.5mm, F.Cu at (119.6, 82.8)
Routing:
- net +3V3_SYS: track 91.5 -> 104.3 mm

Commit message: fix(camera): U6/U7 -> C132016, the reel code that is actually in stock
The first assembly order shipped WITHOUT the two supervisors, leaving them
to be hand-soldered. The cause was not an unobtainable part: the BOM named
C702125 (TLV803SDBZT) and LCSC had zero, so JLCPCB simply dropped the line.

C132016 is TLV803SDBZR -- the same die. In TI's numbering the trailing
T/R is only reel size (250-piece tape vs 3000-piece reel); S is the 2.93 V
threshold variant and DBZ the SOT-23-3 package. Same threshold, same
open-drain RESET, same 200 ms delay, same pinout (1 GND, 2 RESET, 3 VDD).
It is in JLCPCB's assembly library for both Economic and Standard PCBA and
stocked in the thousands, and reel is the format the feeders want anyway.

NOTHING GEOMETRIC CHANGES. The diff to the .kicad_pcb is six (property ...)
lines on F.Fab -- Value, MPN and LCSC on the two footprints. No gerber,
drill or CPL file is touched, so the existing fabrication package stays
valid and the copper is bit-identical. The schematic is updated alongside
the CSV because the BOM regenerates from it (README section 15.6);
editing only the CSV would silently revert.

Also documented in CAMERA_POWER_DESIGN.md section 6, because substituting a
supervisor here has two silent failure modes, both from the TI datasheet
(SBVS157E):

  - TLV853 and TLV863 are functionally identical to the TLV803 but have
    DIFFERENT PINOUTS. "Same family" is precisely the wrong heuristic.
  - TLV809 and TLV810 are push-pull, not open-drain. A push-pull output
    drives U5.EN from its own supply and destroys the vdd_33 interlock that
    section 6 depends on to keep vdd_pix from preceding vdd_33.

Approved alternate recorded: TLV803R (C702124), 2.64 V, same pinout, with
a better false-trip margin (529 mV vs 239 mV) but a later assert point --
flagged as needing the section 7.5 power-down sim re-run before it is
trusted. Of the threshold options only S and R are usable; M (4.38 V) never
releases on a 3.3 V rail.

README section 15.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
Parts:
- U6, U7: value TLV803SDBZT -> TLV803SDBZR
Changed lines of the file:
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@@
 			)
 		)
-		(property "Value" "TLV803SDBZT"
+		(property "Value" "TLV803SDBZR"
 			(at 0 2.4 0)
 			(layer "F.Fab")
@@
 			)
 		)
-		(property "MPN" "TLV803SDBZT"
+		(property "MPN" "TLV803SDBZR"
 			(at 0 0 0)
 			(unlocked yes)
@@
 			)
 		)
-		(property "LCSC" "C702125"
+		(property "LCSC" "C132016"
 			(at 0 0 0)
 			(unlocked yes)
@@
 			)
 		)
-		(property "Value" "TLV803SDBZT"
+		(property "Value" "TLV803SDBZR"
 			(at 0 2.4 0)
 			(layer "F.Fab")
@@
 			)
 		)
-		(property "MPN" "TLV803SDBZT"
+		(property "MPN" "TLV803SDBZR"
 			(at 0 0 0)
 			(unlocked yes)
@@
 			)
 		)
-		(property "LCSC" "C702125"
+		(property "LCSC" "C132016"
 			(at 0 0 0)
 			(unlocked yes)
