File: LauEsp32Config_Pt_Stack/LauEsp32Config_Pt_Stack.kicad_sch (KiCad schematic)
At the start: 58 parts, among them J1 DF40 Bank A (BOTTOM, plug), J2 DF40 Bank B (BOTTOM, plug), J3 DF40 Control (BOTTOM, plug), J4 DF40 Bank A (TOP, receptacle), J5 DF40 Bank B (TOP, receptacle), J6 DF40 Control (TOP, receptacle), J7 microSD Molex 104031-0811, Q1 2N7002, Q2 2N7002, U1 ESP32-S3-MINI-1U-N8, U2 SN74LVC125APWR

Commit message: feat(esp32-card): JTAG straps to 0R, JLCPCB upload set as ordered 2026-09-30 -- ORDERED
TCK/TMS/TDI straps R10-R12 (and rev B R14-R16) 33R -> 0R, C17168. The Pt isolates its
FT2232H with only 100R (RN2); with 33R here an ESP32 pulling low against an FTDI still
driving high (left in MPSSE by a loader run) reaches ~0.8 V at the FPGA -- VIL(max). 0R
gives ~0.3-0.4 V. TDO straps R13/R17 are received, not driven: stay 33R. Changed in
gen_schematic.py and regenerated (sch + both BOMs); the unmodified generator was first
shown to reproduce the committed files byte for byte. Board: Value and LCSC fields only.
Parity back to the 58 metadata-only MPN/LCSC warnings; DRC 0 / 0 unconnected; ERC 0.

gen_schematic.py finds KiCad under either machine's install path.

production/jlcpcb/ is exactly what was uploaded: gerbers (KiCad 10.0.3, generated twice,
identical but for timestamps, zip verified byte for byte), BOM (46 placements, 4 DNP
excluded, all 17 lines in stock), and a CPL with rotations corrected to JLC's library:
Q1/Q2 180 -> 0, U2 0 -> 270, J7 90 -> 270, found by fitting each LCSC part's EasyEDA
footprint to the KiCad one.

Pre-order review, four independent checks, no blocker: U1 land pattern and all 65 pins
vs the S3-MINI-1U datasheet; J1-J6 vs Alchitry's official V2 element library (positions,
genders, 210-pad pass-through); JTAG / PROGRAM_B / DONE / microSD / power vs the Pt Rev A
schematic; JLC DFM limits. Order: Single PCB (JLC adds rails), ENIG, 0.2 mm vias
(TG155 + Kelvin forced), Epoxy Filled & Capped for the 141 vias at or in pads.

README: status (layout routed, fab ordered), 8.1 order record, 6.0 pad table rewritten
for the S3 as built (it still described the C3), 4.2 strap-voltage note.
SCHEMATIC.md: strap values and BOM table.

Co-Authored-By: Claude Opus 5.5 <noreply@anthropic.com>
Parts:
- R10, R11, R12, R14, R15, R16: value 33R -> 0R; LCSC C25105 -> C17168; MPN 0402WGF330JTCE -> 0402WGF0000TCE
Changed lines of the file:
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@@
 			)
 		)
-		(property "Value" "33R"
+		(property "Value" "0R"
 			(at 480.06 209.55 0)
 			(effects
@@
 			)
 		)
-		(property "LCSC" "C25105"
+		(property "LCSC" "C17168"
 			(at 477.52 208.28 0)
 			(hide yes)
@@
 			)
 		)
-		(property "MPN" "0402WGF330JTCE"
+		(property "MPN" "0402WGF0000TCE"
 			(at 477.52 208.28 0)
 			(hide yes)
@@
 			)
 		)
-		(property "Value" "33R"
+		(property "Value" "0R"
 			(at 492.76 209.55 0)
 			(effects
@@
 			)
 		)
-		(property "LCSC" "C25105"
+		(property "LCSC" "C17168"
 			(at 490.22 208.28 0)
 			(hide yes)
@@
 			)
 		)
-		(property "MPN" "0402WGF330JTCE"
+		(property "MPN" "0402WGF0000TCE"
 			(at 490.22 208.28 0)
 			(hide yes)
@@
 			)
 		)
-		(property "Value" "33R"
+		(property "Value" "0R"
 			(at 505.46 209.55 0)
 			(effects
@@
 			)
 		)
-		(property "LCSC" "C25105"
+		(property "LCSC" "C17168"
 			(at 502.92 208.28 0)
 			(hide yes)
@@
 			)
 		)
-		(property "MPN" "0402WGF330JTCE"
+		(property "MPN" "0402WGF0000TCE"
 			(at 502.92 208.28 0)
 			(hide yes)
@@
 			)
 		)
-		(property "Value" "33R"
+		(property "Value" "0R"
 			(at 530.86 209.55 0)
 			(effects
@@
 			)
 		)
-		(property "LCSC" "C25105"
+		(property "LCSC" "C17168"
 			(at 528.32 208.28 0)
 			(hide yes)
@@
 			)
 		)
-		(property "MPN" "0402WGF330JTCE"
+		(property "MPN" "0402WGF0000TCE"
 			(at 528.32 208.28 0)
 			(hide yes)
@@
 			)
 		)
-		(property "Value" "33R"
+		(property "Value" "0R"
 			(at 543.56 209.55 0)
 			(effects
@@
 			)
 		)
-		(property "LCSC" "C25105"
+		(property "LCSC" "C17168"
 			(at 541.02 208.28 0)
 			(hide yes)
@@
 			)
 		)
-		(property "MPN" "0402WGF330JTCE"
+		(property "MPN" "0402WGF0000TCE"
 			(at 541.02 208.28 0)
 			(hide yes)
@@
 			)
 		)
-		(property "Value" "33R"
+		(property "Value" "0R"
 			(at 556.26 209.55 0)
 			(effects
@@
 			)
 		)
-		(property "LCSC" "C25105"
+		(property "LCSC" "C17168"
 			(at 553.72 208.28 0)
 			(hide yes)
@@
 			)
 		)
-		(property "MPN" "0402WGF330JTCE"
+		(property "MPN" "0402WGF0000TCE"
 			(at 553.72 208.28 0)
 			(hide yes)
